File: zendrive.sch (KiCad schematic (older format))
At the start: 32 parts, among them CON1 BARREL_JACK, J1 JACK_INPUT, J2 JACK_OUTPUT, Q1 2N7000, Q2 2N7000, SW1 3PDT, U1 OPA2604

Commit message: Update
Parts:
- C1: footprint (none) -> Capacitors_SMD:c_elec_6.3x5.3
- C2: footprint (none) -> Capacitors_SMD:c_elec_5x5.3
- C3, C5, C6, C7: footprint (none) -> Capacitors_ThroughHole:Capacitor7.5MMDiscRM5
- C4: footprint (none) -> Capacitors_ThroughHole:Capacitor3MMDiscRM2.5
- CON1: footprint (none) -> Connect:BARREL_JACK
- D1, D2, D3: footprint (none) -> Diodes_ThroughHole:Diode_DO-35_SOD27_Horizontal_RM10
- D4: footprint (none) -> Diodes_ThroughHole:Diode_LED_5mm_round_vertical
- Q1, Q2: footprint Discret:TO92 -> Housings_TO-92:TO-92-FET-inline-narrow-oval-SGD
- R1, R2, R3, R4, R5, R6, R7, R8, R9: footprint (none) -> Resistors_SMD:R_1206_HandSoldering
- SW1: footprint (none) -> zendrive:3PDT
- U1: footprint (none) -> Sockets_DIP:DIP-8__300_ELL
Changed lines of the file:
@@
 F 0 "U1" H 3600 5650 60  0000 C CNN
 F 1 "OPA2604" H 3650 5300 60  0000 C CNN
-F 2 "" H 3450 5500 60  0001 C CNN
+F 2 "Sockets_DIP:DIP-8__300_ELL" H 3450 5500 60  0001 C CNN
 F 3 "" H 3450 5500 60  0000 C CNN
 	1    3450 5500
@@
 F 0 "U1" H 7000 5650 60  0000 C CNN
 F 1 "OPA2604" H 7050 5300 60  0000 C CNN
-F 2 "" H 6850 5500 60  0001 C CNN
+F 2 "Sockets_DIP:DIP-8__300_ELL" H 6850 5500 60  0001 C CNN
 F 3 "" H 6850 5500 60  0000 C CNN
 	2    6850 5500
@@
 F 0 "C1" H 1450 1550 40  0000 L CNN
 F 1 "100uF" H 1456 1365 40  0000 L CNN
-F 2 "" H 1488 1300 30  0001 C CNN
+F 2 "Capacitors_SMD:c_elec_6.3x5.3" H 1488 1300 30  0001 C CNN
 F 3 "" H 1450 1450 60  0000 C CNN
 	1    1450 1450
@@
 F 0 "C2" H 2400 1800 40  0000 L CNN
 F 1 "47uF" H 2406 1615 40  0000 L CNN
-F 2 "" H 2438 1550 30  0001 C CNN
+F 2 "Capacitors_SMD:c_elec_5x5.3" H 2438 1550 30  0001 C CNN
 F 3 "" H 2400 1700 60  0000 C CNN
 	1    2400 1700
@@
 F 0 "R1" V 2030 1100 40  0000 C CNN
 F 1 "10K" V 1957 1101 40  0000 C CNN
-F 2 "" V 1880 1100 30  0001 C CNN
+F 2 "Resistors_SMD:R_1206_HandSoldering" V 1880 1100 30  0001 C CNN
 F 3 "" H 1950 1100 30  0000 C CNN
 	1    1950 1100
@@
 F 0 "R2" V 2030 1700 40  0000 C CNN
 F 1 "10K" V 1957 1701 40  0000 C CNN
-F 2 "" V 1880 1700 30  0001 C CNN
+F 2 "Resistors_SMD:R_1206_HandSoldering" V 1880 1700 30  0001 C CNN
 F 3 "" H 1950 1700 30  0000 C CNN
 	1    1950 1700
@@
 F 0 "CON1" H 7650 1500 60  0000 C CNN
 F 1 "BARREL_JACK" H 7650 1050 60  0000 C CNN
-F 2 "" H 7650 1250 60  0001 C CNN
+F 2 "Connect:BARREL_JACK" H 7650 1250 60  0001 C CNN
 F 3 "" H 7650 1250 60  0000 C CNN
 	1    7650 1250
@@
 F 0 "C5" H 1950 3650 40  0000 L CNN
 F 1 "100nF" H 1956 3465 40  0000 L CNN
-F 2 "" H 1988 3400 30  0001 C CNN
+F 2 "Capacitors_ThroughHole:Capacitor7.5MMDiscRM5" H 1988 3400 30  0001 C CNN
 F 3 "" H 1950 3550 60  0000 C CNN
 	1    1950 3550
@@
 F 0 "R7" V 2030 4900 40  0000 C CNN
 F 1 "1K" V 1957 4901 40  0000 C CNN
-F 2 "" V 1880 4900 30  0001 C CNN
+F 2 "Resistors_SMD:R_1206_HandSoldering" V 1880 4900 30  0001 C CNN
 F 3 "" H 1950 4900 30  0000 C CNN
 	1    1950 4900
@@
 F 0 "C6" V 1800 5650 40  0000 L CNN
 F 1 "470nF" V 1800 5350 40  0000 L CNN
-F 2 "" H 1788 5450 30  0001 C CNN
+F 2 "Capacitors_ThroughHole:Capacitor7.5MMDiscRM5" H 1788 5450 30  0001 C CNN
 F 3 "" H 1750 5600 60  0000 C CNN
 	1    1750 5600
@@
 F 0 "R6" V 1430 6100 40  0000 C CNN
 F 1 "2M" V 1357 6101 40  0000 C CNN
-F 2 "" V 1280 6100 30  0001 C CNN
+F 2 "Resistors_SMD:R_1206_HandSoldering" V 1280 6100 30  0001 C CNN
 F 3 "" H 1350 6100 30  0000 C CNN
 	1    1350 6100
@@
 F 0 "R5" V 2430 6100 40  0000 C CNN
 F 1 "470K" V 2357 6101 40  0000 C CNN
-F 2 "" V 2280 6100 30  0001 C CNN
+F 2 "Resistors_SMD:R_1206_HandSoldering" V 2280 6100 30  0001 C CNN
 F 3 "" H 2350 6100 30  0000 C CNN
 	1    2350 6100
@@
 F 0 "Q2" V 2950 3351 40  0000 R CNN
 F 1 "2N7000" V 3150 3700 40  0000 R CNN
-F 2 "Discret:TO92" V 2900 3650 29  0000 C CNN
+F 2 "Housings_TO-92:TO-92-FET-inline-narrow-oval-SGD" V 2900 3650 29  0000 C CNN
 F 3 "" H 2950 3500 60  0000 C CNN
 	1    2950 3500
@@
 F 0 "Q1" V 3750 4200 40  0000 R CNN
 F 1 "2N7000" V 3750 4050 40  0000 R CNN
-F 2 "Discret:TO92" V 3500 4200 29  0000 C CNN
+F 2 "Housings_TO-92:TO-92-FET-inline-narrow-oval-SGD" V 3500 4200 29  0000 C CNN
 F 3 "" H 3550 4050 60  0000 C CNN
 	1    3550 4050
@@
 F 0 "D1" H 3400 3500 40  0000 C CNN
 F 1 "BAT41" H 3400 3300 40  0000 C CNN
-F 2 "" H 3400 3400 60  0001 C CNN
+F 2 "Diodes_ThroughHole:Diode_DO-35_SOD27_Horizontal_RM10" H 3400 3400 60  0001 C CNN
 F 3 "" H 3400 3400 60  0000 C CNN
 	1    3400 3400
@@
 F 0 "D2" H 3850 3500 40  0000 C CNN
 F 1 "BAT41" H 3850 3300 40  0000 C CNN
-F 2 "" H 3850 3400 60  0001 C CNN
+F 2 "Diodes_ThroughHole:Diode_DO-35_SOD27_Horizontal_RM10" H 3850 3400 60  0001 C CNN
 F 3 "" H 3850 3400 60  0000 C CNN
 	1    3850 3400
@@
 F 0 "D3" H 3000 4250 40  0000 C CNN
 F 1 "BAT41" H 3000 4050 40  0000 C CNN
-F 2 "" H 3000 4150 60  0001 C CNN
+F 2 "Diodes_ThroughHole:Diode_DO-35_SOD27_Horizontal_RM10" H 3000 4150 60  0001 C CNN
 F 3 "" H 3000 4150 60  0000 C CNN
 	1    3000 4150
@@
 F 0 "C7" V 3400 4650 40  0000 L CNN
 F 1 "100pF" V 3400 4350 40  0000 L CNN
-F 2 "" H 3388 4450 30  0001 C CNN
+F 2 "Capacitors_ThroughHole:Capacitor7.5MMDiscRM5" H 3388 4450 30  0001 C CNN
 F 3 "" H 3350 4600 60  0000 C CNN
 	1    3350 4600
@@
 F 0 "R8" V 3780 2500 40  0000 C CNN
 F 1 "1K" V 3707 2501 40  0000 C CNN
-F 2 "" V 3630 2500 30  0001 C CNN
+F 2 "Resistors_SMD:R_1206_HandSoldering" V 3630 2500 30  0001 C CNN
 F 3 "" H 3700 2500 30  0000 C CNN
 	1    3700 2500
@@
 F 0 "R4" V 4780 5500 40  0000 C CNN
 F 1 "10K" V 4707 5501 40  0000 C CNN
-F 2 "" V 4630 5500 30  0001 C CNN
+F 2 "Resistors_SMD:R_1206_HandSoldering" V 4630 5500 30  0001 C CNN
 F 3 "" H 4700 5500 30  0000 C CNN
 	1    4700 5500
@@
 F 0 "C4" H 5750 6200 40  0000 L CNN
 F 1 "3.3nF" H 5756 6015 40  0000 L CNN
-F 2 "" H 5788 5950 30  0001 C CNN
+F 2 "Capacitors_ThroughHole:Capacitor3MMDiscRM2.5" H 5788 5950 30  0001 C CNN
 F 3 "" H 5750 6100 60  0000 C CNN
 	1    5750 6100
@@
 F 0 "C3" V 7750 5550 40  0000 L CNN
 F 1 "470nF" V 7900 5550 40  0000 L CNN
-F 2 "" H 7838 5350 30  0001 C CNN
+F 2 "Capacitors_ThroughHole:Capacitor7.5MMDiscRM5" H 7838 5350 30  0001 C CNN
 F 3 "" H 7800 5500 60  0000 C CNN
 	1    7800 5500
@@
 F 0 "R3" V 8480 5500 40  0000 C CNN
 F 1 "1K" V 8407 5501 40  0000 C CNN
-F 2 "" V 8330 5500 30  0001 C CNN
+F 2 "Resistors_SMD:R_1206_HandSoldering" V 8330 5500 30  0001 C CNN
 F 3 "" H 8400 5500 30  0000 C CNN
 	1    8400 5500
@@
 F 0 "SW1" H 6700 3650 60  0000 C CNN
 F 1 "3PDT" H 6200 4450 60  0000 C CNN
-F 2 "" H 6450 3250 60  0001 C CNN
+F 2 "zendrive:3PDT" H 6450 3250 60  0001 C CNN
 F 3 "" H 6450 3250 60  0000 C CNN
 	1    6450 3800
@@
 F 0 "D4" H 7750 3450 50  0000 C CNN
 F 1 "LED" H 7750 3250 50  0000 C CNN
-F 2 "" H 7750 3350 60  0001 C CNN
+F 2 "Diodes_ThroughHole:Diode_LED_5mm_round_vertical" H 7750 3350 60  0001 C CNN
 F 3 "" H 7750 3350 60  0000 C CNN
 	1    7750 3350
@@
 F 0 "R9" V 7230 3350 40  0000 C CNN
 F 1 "1K" V 7157 3351 40  0000 C CNN
-F 2 "" V 7080 3350 30  0001 C CNN
+F 2 "Resistors_SMD:R_1206_HandSoldering" V 7080 3350 30  0001 C CNN
 F 3 "" H 7150 3350 30  0000 C CNN
 	1    7150 3350

Commit message: Update
Parts:
- R9: value 1K -> 470R
Changed lines of the file:
@@
 F 0 "Q2" V 2950 3351 40  0000 R CNN
 F 1 "2N7000" V 3150 3700 40  0000 R CNN
-F 2 "Housings_TO-92:TO-92-FET-inline-narrow-oval-SGD" V 2900 3650 29  0000 C CNN
+F 2 "Housings_TO-92:TO-92-FET-inline-narrow-oval-SGD" V 2900 3650 29  0001 C CNN
 F 3 "" H 2950 3500 60  0000 C CNN
 	1    2950 3500
@@
 F 0 "Q1" V 3750 4200 40  0000 R CNN
 F 1 "2N7000" V 3750 4050 40  0000 R CNN
-F 2 "Housings_TO-92:TO-92-FET-inline-narrow-oval-SGD" V 3500 4200 29  0000 C CNN
+F 2 "Housings_TO-92:TO-92-FET-inline-narrow-oval-SGD" V 3500 4200 29  0001 C CNN
 F 3 "" H 3550 4050 60  0000 C CNN
 	1    3550 4050
@@
 P 7150 3350
 F 0 "R9" V 7230 3350 40  0000 C CNN
-F 1 "1K" V 7157 3351 40  0000 C CNN
+F 1 "470R" V 7157 3351 40  0000 C CNN
 F 2 "Resistors_SMD:R_1206_HandSoldering" V 7080 3350 30  0001 C CNN
 F 3 "" H 7150 3350 30  0000 C CNN

Commit message: Adding PCB
Parts:
- BT1: footprint (none) -> Pin_Headers:Pin_Header_Angled_1x02
- J1, J2: footprint (none) -> Local:NRJ6HF_6MM_ST_JACK
- RV-GAIN-2: renamed from GAIN-RV2; footprint (none) -> Local:POT_HEADER_3
- RV-TONE-3: renamed from TONE-RV3; footprint (none) -> Local:POT_HEADER_3
- RV-VOICE-1: renamed from VOICE-RV1; footprint (none) -> Local:POT_HEADER_3
- RV-VOLUME-4: renamed from VOLUME-RV4; footprint (none) -> Local:POT_HEADER_3
Changed lines of the file:
@@
 F 0 "J1" H 7250 1800 60  0000 C CNN
 F 1 "JACK_INPUT" H 7450 2250 60  0000 C CNN
-F 2 "" H 7600 2000 60  0001 C CNN
+F 2 "Local:NRJ6HF_6MM_ST_JACK" H 7600 2000 60  0001 C CNN
 F 3 "" H 7600 2000 60  0000 C CNN
 	1    7600 2000
@@
 F 0 "BT1" H 6500 1550 50  0000 C CNN
 F 1 "BATTERY" H 6500 1160 50  0000 C CNN
-F 2 "" H 6500 1350 60  0001 C CNN
+F 2 "Pin_Headers:Pin_Header_Angled_1x02" H 6500 1350 60  0001 C CNN
 F 3 "" H 6500 1350 60  0000 C CNN
 	1    6500 1350
@@
 $EndComp
 $Comp
-L POT VOICE-RV1
+L POT RV-VOICE-1
 U 1 1 54AD9D29
 P 1950 4200
-F 0 "VOICE-RV1" H 1950 4100 50  0000 C CNN
+F 0 "RV-VOICE-1" H 1950 4100 50  0000 C CNN
 F 1 "10K" H 1950 4200 50  0000 C CNN
-F 2 "" H 1950 4200 60  0001 C CNN
+F 2 "Local:POT_HEADER_3" H 1950 4200 60  0001 C CNN
 F 3 "" H 1950 4200 60  0000 C CNN
 	1    1950 4200
@@
 V2
 $Comp
-L POT GAIN-RV2
+L POT RV-GAIN-2
 U 1 1 54ADAC20
 P 3200 2800
-F 0 "GAIN-RV2" H 3200 2700 50  0000 C CNN
+F 0 "RV-GAIN-2" H 3200 2700 50  0000 C CNN
 F 1 "500K" H 3200 2800 50  0000 C CNN
-F 2 "" H 3200 2800 60  0001 C CNN
+F 2 "Local:POT_HEADER_3" H 3200 2800 60  0001 C CNN
 F 3 "" H 3200 2800 60  0000 C CNN
 	1    3200 2800
@@
 $EndComp
 $Comp
-L POT TONE-RV3
+L POT RV-TONE-3
 U 1 1 54ADCC06
 P 5350 5500
-F 0 "TONE-RV3" H 5350 5400 50  0000 C CNN
+F 0 "RV-TONE-3" H 5350 5400 50  0000 C CNN
 F 1 "50K" H 5350 5500 50  0000 C CNN
-F 2 "" H 5350 5500 60  0001 C CNN
+F 2 "Local:POT_HEADER_3" H 5350 5500 60  0001 C CNN
 F 3 "" H 5350 5500 60  0000 C CNN
 	1    5350 5500
@@
 $EndComp
 $Comp
-L POT VOLUME-RV4
+L POT RV-VOLUME-4
 U 1 1 54ADDB89
 P 8950 5750
-F 0 "VOLUME-RV4" H 8950 5650 50  0000 C CNN
+F 0 "RV-VOLUME-4" H 8950 5650 50  0000 C CNN
 F 1 "100K" H 8950 5750 50  0000 C CNN
-F 2 "" H 8950 5750 60  0001 C CNN
+F 2 "Local:POT_HEADER_3" H 8950 5750 60  0001 C CNN
 F 3 "" H 8950 5750 60  0000 C CNN
 	1    8950 5750
@@
 F 0 "J2" H 9750 1250 60  0000 C CNN
 F 1 "JACK_OUTPUT" H 9950 1700 60  0000 C CNN
-F 2 "" H 10100 1450 60  0001 C CNN
+F 2 "Local:NRJ6HF_6MM_ST_JACK" H 10100 1450 60  0001 C CNN
 F 3 "" H 10100 1450 60  0000 C CNN
 	1    10100 1450
